Commit message: 2nd

File: src/slatol3d_description/urdf/slatol.urdf.xacro (robot description, xacro)
@@ -1,14 +1,9 @@
 <?xml version="1.0"?>
 <robot name="slatol" xmlns:xacro="http://www.ros.org/wiki/xacro">
-  <xacro:property name="pi" value="3.1415926535897931"/>
-  <xacro:property name="L1" value="0.30" />    <!-- Abduction Link Length -->
-  <xacro:property name="L2" value="0.35" />    <!-- Thigh Length -->
-  <xacro:property name="L3" value="0.35" />    <!-- Calf Length -->
-  <xacro:property name="base_size" value="0.3" />
+  <xacro:property name="L1" value="0.30" />    <xacro:property name="L2" value="0.35" />    <xacro:property name="L3" value="0.35" />    <xacro:property name="base_size" value="0.3" />
   <xacro:property name="link_radius" value="0.03" />
   <material name="Red"><color rgba="0.8 0 0 1"/></material>
   <material name="Blue"><color rgba="0 0 0.8 1"/></material>
   <material name="Black"><color rgba="0 0 0 1"/></material>
-  <!-- Base link (torso/body) - ROOT -->
   <link name="base_link">
     <visual><geometry><box size="${base_size} ${base_size} ${base_size}" /></geometry><material name="Red"/></visual>
@@ -16,5 +11,4 @@
     <inertial><mass value="5.0"/><inertia ixx="0.1" iyy="0.1" izz="0.1" ixy="0" ixz="0" iyz="0"/></inertial>
   </link>
-  <!-- Joint 1: Hip Abduction/Adduction (HAA) - Rotates about X -->
   <joint name="hip_haa_joint" type="revolute">
     <parent link="base_link"/>
@@ -35,5 +29,4 @@
     </transmission>
   </link>
-  <!-- Joint 2: Hip Flextion/Extension (HFE) - Rotates about Y -->
   <joint name="hip_hfe_joint" type="revolute">
     <parent link="abduction_link"/>
@@ -54,5 +47,4 @@
     </transmission>
   </link>
-  <!-- Joint 3: Knee Flextion/Extension (KFE) -->
   <joint name="knee_kfe_joint" type="revolute">
     <parent link="thigh_link"/>
@@ -73,5 +65,4 @@
     </transmission>
   </link>
-  <!-- Final foot link (end-effector) -->
   <joint name="foot_fixed_joint" type="fixed">
     <parent link="calf_link"/>
@@ -84,5 +75,4 @@
      <inertial><mass value="0.1"/><inertia ixx="0.001" iyy="0.001" izz="0.001" ixy="0" ixz="0" iyz="0"/></inertial>
   </link>
-  <!-- Gazebo Fortress: ROS 2 Control Plugin -->
   <gazebo>
     <plugin name="gazebo_ros2_control" filename="libgazebo_ros2_control.so">

Commit message: fall and testcontrol.py

File: src/slatol3d_description/urdf/slatol.urdf.xacro (robot description, xacro)
@@ -1,5 +1,8 @@
 <?xml version="1.0"?>
 <robot name="slatol" xmlns:xacro="http://www.ros.org/wiki/xacro">
-  <xacro:property name="L1" value="0.30" />    <xacro:property name="L2" value="0.35" />    <xacro:property name="L3" value="0.35" />    <xacro:property name="base_size" value="0.3" />
+  <xacro:property name="L1" value="0.30" />
+  <xacro:property name="L2" value="0.35" />
+  <xacro:property name="L3" value="0.35" />
+  <xacro:property name="base_size" value="0.3" />
   <xacro:property name="link_radius" value="0.03" />
   <material name="Red"><color rgba="0.8 0 0 1"/></material>
@@ -16,6 +19,5 @@
     <origin xyz="0 ${-base_size/2} 0" rpy="0 0 0"/>
     <axis xyz="1 0 0"/>
-    <limit lower="-0.78" upper="0.78" effort="10.0" velocity="2.0"/>
-    <dynamics damping="0.1" friction="0.1"/>
+    <limit lower="-0.78" upper="0.78" effort="100.0" velocity="2.0"/>
   </joint>
   <link name="abduction_link">
@@ -23,9 +25,4 @@
     <collision><geometry><cylinder length="${link_radius}" radius="${link_radius}"/></geometry></collision>
     <inertial><mass value="0.2"/><inertia ixx="0.001" iyy="0.001" izz="0.001" ixy="0" ixz="0" iyz="0"/></inertial>
-    <transmission name="haa_trans">
-        <type>transmission_interface/SimpleTransmission</type>
-        <joint name="hip_haa_joint"><hardwareInterface>hardware_interface/PositionJointInterface</hardwareInterface></joint>
-        <actuator name="haa_motor"><mechanicalReduction>1</mechanicalReduction></actuator>
-    </transmission>
   </link>
   <joint name="hip_hfe_joint" type="revolute">
@@ -34,6 +31,5 @@
     <origin xyz="0 0 ${-base_size/2}" rpy="0 0 0"/>
     <axis xyz="0 1 0"/>
-    <limit lower="-1.57" upper="1.57" effort="10.0" velocity="2.0"/>
-    <dynamics damping="0.1" friction="0.1"/>
+    <limit lower="-1.57" upper="1.57" effort="100.0" velocity="2.0"/>
   </joint>
   <link name="thigh_link">
@@ -41,9 +37,4 @@
     <collision><geometry><cylinder length="${L2}" radius="${link_radius}"/></geometry><origin xyz="0 0 ${-L2/2}" rpy="0 0 0"/></collision>
     <inertial><mass value="1.0"/><inertia ixx="0.01" iyy="0.01" izz="0.01" ixy="0" ixz="0" iyz="0"/></inertial>
-    <transmission name="hfe_trans">
-        <type>transmission_interface/SimpleTransmission</type>
-        <joint name="hip_hfe_joint"><hardwareInterface>hardware_interface/PositionJointInterface</hardwareInterface></joint>
-        <actuator name="hfe_motor"><mechanicalReduction>1</mechanicalReduction></actuator>
-    </transmission>
   </link>
   <joint name="knee_kfe_joint" type="revolute">
@@ -52,6 +43,5 @@
     <origin xyz="0 0 ${-L2}" rpy="0 0 0"/>
     <axis xyz="0 1 0"/>
-    <limit lower="-2.0" upper="0.0" effort="10.0" velocity="2.0"/>
-    <dynamics damping="0.1" friction="0.1"/>
+    <limit lower="-2.0" upper="0.0" effort="100.0" velocity="2.0"/>
   </joint>
   <link name="calf_link">
@@ -59,9 +49,4 @@
     <collision><geometry><cylinder length="${L3}" radius="${link_radius}"/></geometry><origin xyz="0 0 ${-L3/2}" rpy="0 0 0"/></collision>
     <inertial><mass value="1.0"/><inertia ixx="0.01" iyy="0.01" izz="0.01" ixy="0" ixz="0" iyz="0"/></inertial>
-    <transmission name="kfe_trans">
-        <type>transmission_interface/SimpleTransmission</type>
-        <joint name="knee_kfe_joint"><hardwareInterface>hardware_interface/PositionJointInterface</hardwareInterface></joint>
-        <actuator name="kfe_motor"><mechanicalReduction>1</mechanicalReduction></actuator>
-    </transmission>
   </link>
   <joint name="foot_fixed_joint" type="fixed">
@@ -75,6 +60,26 @@
      <inertial><mass value="0.1"/><inertia ixx="0.001" iyy="0.001" izz="0.001" ixy="0" ixz="0" iyz="0"/></inertial>
   </link>
+  <ros2_control name="IgnitionSystem" type="system">
+    <hardware>
+      <plugin>ign_ros2_control/IgnitionSystem</plugin>
+    </hardware>
+    <joint name="hip_haa_joint">
+      <command_interface name="position"/>
+      <state_interface name="position"/>
+      <state_interface name="velocity"/>
+    </joint>
+    <joint name="hip_hfe_joint">
+      <command_interface name="position"/>
+      <state_interface name="position"/>
+      <state_interface name="velocity"/>
+    </joint>
+    <joint name="knee_kfe_joint">
+      <command_interface name="position"/>
+      <state_interface name="position"/>
+      <state_interface name="velocity"/>
+    </joint>
+  </ros2_control>
   <gazebo>
-    <plugin name="gazebo_ros2_control" filename="libgazebo_ros2_control.so">
+    <plugin filename="ign_ros2_control-system" name="ign_ros2_control::IgnitionROS2ControlPlugin">
       <parameters>$(find slatol3d_description)/config/slatol_controllers.yaml</parameters>
     </plugin>

Commit message: ui

File: src/slatol3d_description/urdf/slatol.urdf.xacro (robot description, xacro)
@@ -1,12 +1,57 @@
 <?xml version="1.0"?>
 <robot name="slatol" xmlns:xacro="http://www.ros.org/wiki/xacro">
-  <xacro:property name="L1" value="0.30" />
+  <xacro:property name="base_size" value="0.2" />
+  <xacro:property name="L1" value="0.35" />
   <xacro:property name="L2" value="0.35" />
-  <xacro:property name="L3" value="0.35" />
-  <xacro:property name="base_size" value="0.3" />
   <xacro:property name="link_radius" value="0.03" />
   <material name="Red"><color rgba="0.8 0 0 1"/></material>
   <material name="Blue"><color rgba="0 0 0.8 1"/></material>
   <material name="Black"><color rgba="0 0 0 1"/></material>
+  <material name="Grey"><color rgba="0.5 0.5 0.5 0.5"/></material>
+  <link name="world"/>
+  <joint name="world_slide_x" type="prismatic">
+    <parent link="world"/>
+    <child link="virtual_rail_x"/>
+    <origin xyz="0 0 0" rpy="0 0 0"/>
+    <axis xyz="1 0 0"/>
+    <limit lower="-100" upper="100" effort="20000" velocity="100"/>
+    <dynamics damping="0.0" friction="0.0"/>
+  </joint>
+  <link name="virtual_rail_x">
+    <visual>
+        <geometry><box size="5.0 0.05 0.05"/></geometry>
+        <material name="Grey"/>
+    </visual>
+    <inertial>
+        <mass value="2.0"/>
+        <inertia ixx="0.1" iyy="0.1" izz="0.1" ixy="0" ixz="0" iyz="0"/>
+    </inertial>
+  </link>
+  <joint name="world_slide_z" type="prismatic">
+    <parent link="virtual_rail_x"/>
+    <child link="virtual_rail_z"/>
+    <origin xyz="0 0 0" rpy="0 0 0"/>
+    <axis xyz="0 0 1"/>
+    <limit lower="0" upper="50" effort="20000" velocity="100"/>
+    <dynamics damping="0.0" friction="0.0"/>
+  </joint>
+  <link name="virtual_rail_z">
+    <visual>
+        <geometry><box size="0.05 0.05 2.0"/></geometry>
+        <material name="Grey"/>
+    </visual>
+    <inertial>
+        <mass value="2.0"/>
+        <inertia ixx="0.1" iyy="0.1" izz="0.1" ixy="0" ixz="0" iyz="0"/>
+    </inertial>
+  </link>
+  <joint name="boom_pitch" type="revolute">
+    <parent link="virtual_rail_z"/>
+    <child link="base_link"/>
+    <origin xyz="0 0 0" rpy="0 0 0"/>
+    <axis xyz="0 1 0"/>
+    <limit lower="-6.28" upper="6.28" effort="1000" velocity="50"/>
+    <dynamics damping="0.0" friction="0.0"/>
+  </joint>
   <link name="base_link">
     <visual><geometry><box size="${base_size} ${base_size} ${base_size}" /></geometry><material name="Red"/></visual>
@@ -17,11 +62,10 @@
     <parent link="base_link"/>
     <child link="abduction_link"/>
-    <origin xyz="0 ${-base_size/2} 0" rpy="0 0 0"/>
+    <origin xyz="0 0 0" rpy="0 0 0"/>
     <axis xyz="1 0 0"/>
-    <limit lower="-0.78" upper="0.78" effort="100.0" velocity="2.0"/>
+    <limit lower="-0.0" upper="0.0" effort="1000" velocity="0"/>
   </joint>
   <link name="abduction_link">
-    <visual><geometry><cylinder length="${link_radius}" radius="${link_radius}"/></geometry><material name="Blue"/></visual>
-    <collision><geometry><cylinder length="${link_radius}" radius="${link_radius}"/></geometry></collision>
+    <visual><geometry><cylinder length="0.05" radius="${link_radius}"/></geometry><material name="Blue"/></visual>
     <inertial><mass value="0.2"/><inertia ixx="0.001" iyy="0.001" izz="0.001" ixy="0" ixz="0" iyz="0"/></inertial>
   </link>
@@ -29,11 +73,11 @@
     <parent link="abduction_link"/>
     <child link="thigh_link"/>
-    <origin xyz="0 0 ${-base_size/2}" rpy="0 0 0"/>
+    <origin xyz="0 0 0" rpy="0 0 0"/>
     <axis xyz="0 1 0"/>
-    <limit lower="-1.57" upper="1.57" effort="100.0" velocity="2.0"/>
+    <limit lower="-1.57" upper="1.57" effort="100.0" velocity="10.0"/>
   </joint>
   <link name="thigh_link">
-    <visual><geometry><cylinder length="${L2}" radius="${link_radius}"/></geometry><origin xyz="0 0 ${-L2/2}" rpy="0 0 0"/> <material name="Red"/></visual>
-    <collision><geometry><cylinder length="${L2}" radius="${link_radius}"/></geometry><origin xyz="0 0 ${-L2/2}" rpy="0 0 0"/></collision>
+    <visual><geometry><cylinder length="${L1}" radius="${link_radius}"/></geometry><origin xyz="0 0 ${-L1/2}" rpy="0 0 0"/><material name="Grey"/></visual>
+    <collision><geometry><cylinder length="${L1}" radius="${link_radius}"/></geometry><origin xyz="0 0 ${-L1/2}" rpy="0 0 0"/></collision>
     <inertial><mass value="1.0"/><inertia ixx="0.01" iyy="0.01" izz="0.01" ixy="0" ixz="0" iyz="0"/></inertial>
   </link>
@@ -41,11 +85,11 @@
     <parent link="thigh_link"/>
     <child link="calf_link"/>
-    <origin xyz="0 0 ${-L2}" rpy="0 0 0"/>
+    <origin xyz="0 0 ${-L1}" rpy="0 0 0"/>
     <axis xyz="0 1 0"/>
-    <limit lower="-2.0" upper="0.0" effort="100.0" velocity="2.0"/>
+    <limit lower="-2.6" upper="0.0" effort="100.0" velocity="10.0"/>
   </joint>
   <link name="calf_link">
-    <visual><geometry><cylinder length="${L3}" radius="${link_radius}"/></geometry><origin xyz="0 0 ${-L3/2}" rpy="0 0 0"/><material name="Blue"/></visual>
-    <collision><geometry><cylinder length="${L3}" radius="${link_radius}"/></geometry><origin xyz="0 0 ${-L3/2}" rpy="0 0 0"/></collision>
+    <visual><geometry><cylinder length="${L2}" radius="${link_radius}"/></geometry><origin xyz="0 0 ${-L2/2}" rpy="0 0 0"/><material name="Black"/></visual>
+    <collision><geometry><cylinder length="${L2}" radius="${link_radius}"/></geometry><origin xyz="0 0 ${-L2/2}" rpy="0 0 0"/></collision>
     <inertial><mass value="1.0"/><inertia ixx="0.01" iyy="0.01" izz="0.01" ixy="0" ixz="0" iyz="0"/></inertial>
   </link>
@@ -53,30 +97,17 @@
     <parent link="calf_link"/>
     <child link="foot_link"/>
-    <origin xyz="0 0 ${-L3}" rpy="0 0 0"/>
+    <origin xyz="0 0 ${-L2}" rpy="0 0 0"/>
   </joint>
   <link name="foot_link">
-     <visual><geometry><sphere radius="0.05"/></geometry><material name="Black"/></visual>
-     <collision><geometry><sphere radius="0.05"/></geometry></collision>
+     <visual><geometry><sphere radius="0.04"/></geometry><material name="Red"/></visual>
+     <collision><geometry><sphere radius="0.04"/></geometry></collision>
+     <surface><friction><ode><mu>10.0</mu><mu2>10.0</mu2></ode></friction></surface>
      <inertial><mass value="0.1"/><inertia ixx="0.001" iyy="0.001" izz="0.001" ixy="0" ixz="0" iyz="0"/></inertial>
   </link>
   <ros2_control name="IgnitionSystem" type="system">
-    <hardware>
-      <plugin>ign_ros2_control/IgnitionSystem</plugin>
-    </hardware>
-    <joint name="hip_haa_joint">
-      <command_interface name="position"/>
-      <state_interface name="position"/>
-      <state_interface name="velocity"/>
-    </joint>
-    <joint name="hip_hfe_joint">
-      <command_interface name="position"/>
-      <state_interface name="position"/>
-      <state_interface name="velocity"/>
-    </joint>
-    <joint name="knee_kfe_joint">
-      <command_interface name="position"/>
-      <state_interface name="position"/>
-      <state_interface name="velocity"/>
-    </joint>
+    <hardware><plugin>ign_ros2_control/IgnitionSystem</plugin></hardware>
+    <joint name="hip_haa_joint"><command_interface name="position"/><state_interface name="position"/><state_interface name="velocity"/></joint>
+    <joint name="hip_hfe_joint"><command_interface name="position"/><state_interface name="position"/><state_interface name="velocity"/></joint>
+    <joint name="knee_kfe_joint"><command_interface name="position"/><state_interface name="position"/><state_interface name="velocity"/></joint>
   </ros2_control>
   <gazebo>

Commit message: lev

File: src/slatol3d_description/urdf/slatol.urdf.xacro (robot description, xacro)
@@ -15,5 +15,5 @@
     <origin xyz="0 0 0" rpy="0 0 0"/>
     <axis xyz="1 0 0"/>
-    <limit lower="-100" upper="100" effort="20000" velocity="100"/>
+    <limit lower="-100.0" upper="100.0" effort="20000" velocity="100"/>
     <dynamics damping="0.0" friction="0.0"/>
   </joint>
@@ -24,6 +24,5 @@
     </visual>
     <inertial>
-        <mass value="2.0"/>
-        <inertia ixx="0.1" iyy="0.1" izz="0.1" ixy="0" ixz="0" iyz="0"/>
+        <mass value="0.1"/> <inertia ixx="0.01" iyy="0.01" izz="0.01" ixy="0" ixz="0" iyz="0"/>
     </inertial>
   </link>
@@ -33,5 +32,5 @@
     <origin xyz="0 0 0" rpy="0 0 0"/>
     <axis xyz="0 0 1"/>
-    <limit lower="0" upper="50" effort="20000" velocity="100"/>
+    <limit lower="-50.0" upper="50.0" effort="20000" velocity="100"/>
     <dynamics damping="0.0" friction="0.0"/>
   </joint>
@@ -42,6 +41,5 @@
     </visual>
     <inertial>
-        <mass value="2.0"/>
-        <inertia ixx="0.1" iyy="0.1" izz="0.1" ixy="0" ixz="0" iyz="0"/>
+        <mass value="0.1"/> <inertia ixx="0.01" iyy="0.01" izz="0.01" ixy="0" ixz="0" iyz="0"/>
     </inertial>
   </link>

Commit message: add ref

File: src/slatol3d_description/urdf/slatol.urdf.xacro (robot description, xacro)
@@ -15,14 +15,11 @@
     <origin xyz="0 0 0" rpy="0 0 0"/>
     <axis xyz="1 0 0"/>
-    <limit lower="-100.0" upper="100.0" effort="20000" velocity="100"/>
+    <limit lower="-100" upper="100" effort="20000" velocity="100"/>
     <dynamics damping="0.0" friction="0.0"/>
   </joint>
   <link name="virtual_rail_x">
-    <visual>
-        <geometry><box size="5.0 0.05 0.05"/></geometry>
-        <material name="Grey"/>
-    </visual>
     <inertial>
-        <mass value="0.1"/> <inertia ixx="0.01" iyy="0.01" izz="0.01" ixy="0" ixz="0" iyz="0"/>
+        <mass value="0.01"/>
+        <inertia ixx="0.0001" iyy="0.0001" izz="0.0001" ixy="0" ixz="0" iyz="0"/>
     </inertial>
   </link>
@@ -32,14 +29,11 @@
     <origin xyz="0 0 0" rpy="0 0 0"/>
     <axis xyz="0 0 1"/>
-    <limit lower="-50.0" upper="50.0" effort="20000" velocity="100"/>
+    <limit lower="-10" upper="50" effort="20000" velocity="100"/>
     <dynamics damping="0.0" friction="0.0"/>
   </joint>
   <link name="virtual_rail_z">
-    <visual>
-        <geometry><box size="0.05 0.05 2.0"/></geometry>
-        <material name="Grey"/>
-    </visual>
     <inertial>
-        <mass value="0.1"/> <inertia ixx="0.01" iyy="0.01" izz="0.01" ixy="0" ixz="0" iyz="0"/>
+        <mass value="0.01"/>
+        <inertia ixx="0.0001" iyy="0.0001" izz="0.0001" ixy="0" ixz="0" iyz="0"/>
     </inertial>
   </link>
@@ -56,4 +50,10 @@
     <collision><geometry><box size="${base_size} ${base_size} ${base_size}" /></geometry></collision>
     <inertial><mass value="5.0"/><inertia ixx="0.1" iyy="0.1" izz="0.1" ixy="0" ixz="0" iyz="0"/></inertial>
+    <sensor name="imu_sensor" type="imu">
+      <always_on>1</always_on>
+      <update_rate>100</update_rate>
+      <visualize>true</visualize>
+      <topic>imu</topic>
+    </sensor>
   </link>
   <joint name="hip_haa_joint" type="revolute">
@@ -62,5 +62,5 @@
     <origin xyz="0 0 0" rpy="0 0 0"/>
     <axis xyz="1 0 0"/>
-    <limit lower="-0.0" upper="0.0" effort="1000" velocity="0"/>
+    <limit lower="-0.5" upper="0.5" effort="1000" velocity="20"/>
   </joint>
   <link name="abduction_link">
@@ -73,5 +73,5 @@
     <origin xyz="0 0 0" rpy="0 0 0"/>
     <axis xyz="0 1 0"/>
-    <limit lower="-1.57" upper="1.57" effort="100.0" velocity="10.0"/>
+    <limit lower="-1.57" upper="1.57" effort="200.0" velocity="20.0"/>
   </joint>
   <link name="thigh_link">
@@ -85,5 +85,5 @@
     <origin xyz="0 0 ${-L1}" rpy="0 0 0"/>
     <axis xyz="0 1 0"/>
-    <limit lower="-2.6" upper="0.0" effort="100.0" velocity="10.0"/>
+    <limit lower="-2.6" upper="0.0" effort="200.0" velocity="20.0"/>
   </joint>
   <link name="calf_link">
@@ -100,5 +100,5 @@
      <visual><geometry><sphere radius="0.04"/></geometry><material name="Red"/></visual>
      <collision><geometry><sphere radius="0.04"/></geometry></collision>
-     <surface><friction><ode><mu>10.0</mu><mu2>10.0</mu2></ode></friction></surface>
+     <surface><friction><ode><mu>100.0</mu><mu2>100.0</mu2></ode></friction></surface>
      <inertial><mass value="0.1"/><inertia ixx="0.001" iyy="0.001" izz="0.001" ixy="0" ixz="0" iyz="0"/></inertial>
   </link>
@@ -113,4 +113,6 @@
       <parameters>$(find slatol3d_description)/config/slatol_controllers.yaml</parameters>
     </plugin>
+    <plugin filename="libignition-gazebo-imu-system.so" name="ignition::gazebo::systems::Imu">
+    </plugin>
   </gazebo>
 </robot>

Commit message: error

File: src/slatol3d_description/urdf/slatol.urdf.xacro (robot description, xacro)
@@ -56,4 +56,13 @@
       <topic>imu</topic>
     </sensor>
+    <sensor name="lidar_sensor" type="gpu_lidar">
+        <pose>0 0 0 0 1.57 0</pose> <visualize>true</visualize>
+        <update_rate>50</update_rate>
+        <topic>slatol/lidar</topic>
+        <ray>
+            <scan><horizontal><samples>1</samples><resolution>1</resolution><min_angle>0</min_angle><max_angle>0</max_angle></horizontal></scan>
+            <range><min>0.05</min><max>10.0</max><resolution>0.01</resolution></range>
+        </ray>
+    </sensor>
   </link>
   <joint name="hip_haa_joint" type="revolute">
@@ -99,7 +108,17 @@
   <link name="foot_link">
      <visual><geometry><sphere radius="0.04"/></geometry><material name="Red"/></visual>
-     <collision><geometry><sphere radius="0.04"/></geometry></collision>
-     <surface><friction><ode><mu>100.0</mu><mu2>100.0</mu2></ode></friction></surface>
+     <collision>
+        <geometry><sphere radius="0.04"/></geometry>
+        <surface><friction><ode><mu>1.0</mu><mu2>1.0</mu2></ode></friction></surface>
+     </collision>
      <inertial><mass value="0.1"/><inertia ixx="0.001" iyy="0.001" izz="0.001" ixy="0" ixz="0" iyz="0"/></inertial>
+     <sensor name="foot_contact" type="contact">
+        <update_rate>1000</update_rate>
+        <always_on>1</always_on>
+        <contact>
+            <collision>foot_link_fixed_joint_lump__foot_link_collision_1</collision>
+        </contact>
+        <topic>slatol/contact</topic>
+     </sensor>
   </link>
   <ros2_control name="IgnitionSystem" type="system">
@@ -113,5 +132,8 @@
       <parameters>$(find slatol3d_description)/config/slatol_controllers.yaml</parameters>
     </plugin>
-    <plugin filename="libignition-gazebo-imu-system.so" name="ignition::gazebo::systems::Imu">
+    <plugin filename="libignition-gazebo-imu-system.so" name="ignition::gazebo::systems::Imu"></plugin>
+    <plugin filename="libignition-gazebo-contact-system.so" name="ignition::gazebo::systems::Contact"></plugin>
+    <plugin filename="libignition-gazebo-sensors-system.so" name="ignition::gazebo::systems::Sensors">
+        <render_engine>ogre2</render_engine>
     </plugin>
   </gazebo>
